Commit message: Added material color

File: navigator_description/urdf/navigator_description.urdf (robot description, URDF)
Before this commit: robot robotr_description, 21 links, 20 joints
Links:
- link 4cm_studs: geometry collision mesh filename=package://navigator_description/meshes/4cm_studs.STL; visual mesh filename=package://navigator_description/meshes/4cm_studs.STL
- link 6cm_studs: geometry collision mesh filename=package://navigator_description/meshes/6cm_studs.STL; visual mesh filename=package://navigator_description/meshes/6cm_studs.STL
- link base_link: geometry collision mesh filename=package://navigator_description/meshes/base_link.STL; visual mesh filename=package://navigator_description/meshes/base_link.STL
- link black_plate_big: geometry collision mesh filename=package://navigator_description/meshes/black_plate_big.STL; visual mesh filename=package://navigator_description/meshes/black_plate_big.STL
- link black_plate_small: geometry collision mesh filename=package://navigator_description/meshes/black_plate_small.STL; visual mesh filename=package://navigator_description/meshes/black_plate_small.STL
- link castor: geometry collision mesh filename=package://navigator_description/meshes/castor.STL; visual mesh filename=package://navigator_description/meshes/castor.STL
- link castor_base: geometry collision mesh filename=package://navigator_description/meshes/castor_base.STL; visual mesh filename=package://navigator_description/meshes/castor_base.STL
- link castor_studs: geometry collision mesh filename=package://navigator_description/meshes/castor_studs.STL; visual mesh filename=package://navigator_description/meshes/castor_studs.STL
- link kinect: geometry collision mesh filename=package://navigator_description/meshes/kinect.STL; visual mesh filename=package://navigator_description/meshes/kinect.STL
- link l_clamp: geometry collision mesh filename=package://navigator_description/meshes/l_clamp.STL; visual mesh filename=package://navigator_description/meshes/l_clamp.STL
- link l_motor: geometry collision mesh filename=package://navigator_description/meshes/l_motor.STL; visual mesh filename=package://navigator_description/meshes/l_motor.STL
- link l_rim: geometry collision mesh filename=package://navigator_description/meshes/l_rim.STL; visual mesh filename=package://navigator_description/meshes/l_rim.STL
- link l_shaft: geometry collision mesh filename=package://navigator_description/meshes/l_shaft.STL; visual mesh filename=package://navigator_description/meshes/l_shaft.STL
- link l_wheel: geometry collision mesh filename=package://navigator_description/meshes/l_wheel.STL; visual mesh filename=package://navigator_description/meshes/l_wheel.STL
- link r_clamp: geometry collision mesh filename=package://navigator_description/meshes/r_clamp.STL; visual mesh filename=package://navigator_description/meshes/r_clamp.STL
- link r_motor: geometry collision mesh filename=package://navigator_description/meshes/r_motor.STL; visual mesh filename=package://navigator_description/meshes/r_motor.STL
- link r_rim: geometry collision mesh filename=package://navigator_description/meshes/r_rim.STL; visual mesh filename=package://navigator_description/meshes/r_rim.STL
- link r_shaft: geometry collision mesh filename=package://navigator_description/meshes/r_shaft.STL; visual mesh filename=package://navigator_description/meshes/r_shaft.STL
- link r_wheel: geometry collision mesh filename=package://navigator_description/meshes/r_wheel.STL; visual mesh filename=package://navigator_description/meshes/r_wheel.STL
- link upper_plate: geometry collision mesh filename=package://navigator_description/meshes/upper_plate.STL; visual mesh filename=package://navigator_description/meshes/upper_plate.STL
Joints:
- joint base_joint: origin xyz=0 0 0.07 rpy=0 0 0 -> xyz=0 0 0.063 rpy=0 0 0
